File: Radio_Receiver_McCormick_Mendoza/Display.kicad_sch (KiCad schematic)
At the start: 0 parts

Commit message: Merge conflict resolution.
Other:
- title: (none) -> Radio Receiver
Changed lines of the file:
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@@
 	(paper "A4")
 	(title_block
+		(title "Radio Receiver")
 		(date "2026-04-19")
 		(rev "0.0.1")

Commit message: Propogated Title Block Fields
Other:
- company: (none) -> Walla Walla University
Changed lines of the file:
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@@
 		(date "2026-04-19")
 		(rev "0.0.1")
+		(company "Walla Walla University")
 		(comment 2 "Daniel Mendoza")
 		(comment 3 "Jeffrey McCormick")

Commit message: Schematic edits power and signal systems
Parts:
- added J25: OLED, Connector_PinSocket_2.54mm:PinSocket_1x04_P2.54mm_Vertical, symbol Connector_Generic:Conn_01x04
Connections:
- new net +3.3V: J25.2 (Pin_2)
- new net GND: J25.1 (Pin_1)
- new net SCL: J25.3 (Pin_3)
- new net SDA: J25.4 (Pin_4)
Other:
- note added: "Be careful! Some OLEDs have Vcc and GND swapped! These are in the order GND-Vcc-SCL-SDA."
