File: Radio_Receiver_McCormick_Mendoza/Audio_DAC.kicad_sch (KiCad schematic)
At the start: 46 parts, among them J35 3.5mm_Jack, J38 DAC_FLT, J40 DAC_FMT, J46 3.5mm_Jack, U14 PCM5102A

Commit message: Added MicroSD card and verified footprints
Parts:
- C49: Manufacturer Murata Electronics -> (none)
- C59, C68, C85, C86, C89: Manufacturer AVX -> (none)
- JP10, JP6: footprint (none) -> Jumper:SolderJumper-2_P1.3mm_Bridged_RoundedPad1.0x1.5mm
- R32, R33, R42, R44, R45, R48, R6: Manufacturer UNI-ROYAL(Uniroyal Elec) -> (none)
Changed lines of the file:
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@@
 			)
 		)
-		(property "Manufacturer" "UNI-ROYAL(Uniroyal Elec)"
-			(at 77.47 54.61 0)
-			(hide yes)
-			(show_name no)
-			(do_not_autoplace no)
-			(effects
-				(font
-					(size 1.27 1.27)
-				)
-			)
-		)
 		(property "Part" "0805W8F220KT5E"
 			(at 77.47 54.61 0)
@@
 			)
 		)
-		(property "Manufacturer" "Murata Electronics"
-			(at 177.8 73.66 0)
-			(hide yes)
-			(show_name no)
-			(do_not_autoplace no)
-			(effects
-				(font
-					(size 1.27 1.27)
-				)
-			)
-		)
 		(property "Part" "GRM21BR61H106KE43L"
 			(at 177.8 73.66 0)
@@
 			)
 		)
-		(property "Manufacturer" "UNI-ROYAL(Uniroyal Elec)"
-			(at 182.88 60.96 0)
-			(hide yes)
-			(show_name no)
-			(do_not_autoplace no)
-			(effects
-				(font
-					(size 1.27 1.27)
-				)
-			)
-		)
 		(property "Part" "0603WAF4702T5E"
 			(at 182.88 60.96 0)
@@
 			)
 		)
-		(property "Manufacturer" "AVX"
-			(at 218.44 76.2 0)
-			(hide yes)
-			(show_name no)
-			(do_not_autoplace no)
-			(effects
-				(font
-					(size 1.27 1.27)
-				)
-			)
-		)
 		(property "Part" "TAJB107K006RNJ"
 			(at 218.44 76.2 0)
@@
 			)
 		)
-		(property "Manufacturer" "UNI-ROYAL(Uniroyal Elec)"
-			(at 152.4 85.09 0)
-			(hide yes)
-			(show_name no)
-			(do_not_autoplace no)
-			(effects
-				(font
-					(size 1.27 1.27)
-				)
-			)
-		)
 		(property "Part" "0805W8F1002T5E"
 			(at 152.4 85.09 0)
@@
 			)
 		)
-		(property "Manufacturer" "UNI-ROYAL(Uniroyal Elec)"
-			(at 170.18 77.47 0)
-			(hide yes)
-			(show_name no)
-			(do_not_autoplace no)
-			(effects
-				(font
-					(size 1.27 1.27)
-				)
-			)
-		)
 		(property "Part" "0603WAF6801T5E"
 			(at 170.18 77.47 0)
@@
 			)
 		)
-		(property "Footprint" ""
+		(property "Footprint" "Jumper:SolderJumper-2_P1.3mm_Bridged_RoundedPad1.0x1.5mm"
 			(at 59.69 133.35 0)
 			(hide yes)
@@
 			)
 		)
-		(property "Manufacturer" "AVX"
-			(at 222.25 73.66 0)
-			(hide yes)
-			(show_name no)
-			(do_not_autoplace no)
-			(effects
-				(font
-					(size 1.27 1.27)
-				)
-			)
-		)
 		(property "Part" "TAJB107K006RNJ"
 			(at 222.25 73.66 0)
@@
 			)
 		)
-		(property "Manufacturer" "UNI-ROYAL(Uniroyal Elec)"
-			(at 142.24 85.09 0)
-			(hide yes)
-			(show_name no)
-			(do_not_autoplace no)
-			(effects
-				(font
-					(size 1.27 1.27)
-				)
-			)
-		)
 		(property "Part" "0805W8F1002T5E"
 			(at 142.24 85.09 0)
@@
 			)
 		)
-		(property "Manufacturer" "AVX"
-			(at 229.87 68.58 0)
-			(hide yes)
-			(show_name no)
-			(do_not_autoplace no)
-			(effects
-				(font
-					(size 1.27 1.27)
-				)
-			)
-		)
 		(property "Part" "TAJB107K006RNJ"
 			(at 229.87 68.58 0)
@@
 			)
 		)
-		(property "Footprint" ""
+		(property "Footprint" "Jumper:SolderJumper-2_P1.3mm_Bridged_RoundedPad1.0x1.5mm"
 			(at 33.02 109.22 0)
 			(hide yes)
@@
 			)
 		)
-		(property "Manufacturer" "AVX"
-			(at 226.06 71.12 0)
-			(hide yes)
-			(show_name no)
-			(do_not_autoplace no)
-			(effects
-				(font
-					(size 1.27 1.27)
-				)
-			)
-		)
 		(property "Part" "TAJB107K006RNJ"
 			(at 226.06 71.12 0)
@@
 			)
 		)
-		(property "Manufacturer" "AVX"
-			(at 233.68 66.04 0)
-			(hide yes)
-			(show_name no)
-			(do_not_autoplace no)
-			(effects
-				(font
-					(size 1.27 1.27)
-				)
-			)
-		)
 		(property "Part" "TAJB107K006RNJ"
 			(at 233.68 66.04 0)
@@
 			)
 		)
-		(property "Manufacturer" "UNI-ROYAL(Uniroyal Elec)"
-			(at 242.57 76.2 0)
-			(hide yes)
-			(show_name no)
-			(do_not_autoplace no)
-			(effects
-				(font
-					(size 1.27 1.27)
-				)
-			)
-		)
 		(property "Part" "0805W8F330JT5E"
 			(at 242.57 76.2 0)
@@
 			(at 72.39 54.61 0)
 			(hide yes)
-			(show_name no)
-			(do_not_autoplace no)
-			(effects
-				(font
-					(size 1.27 1.27)
-				)
-			)
-		)
-		(property "Manufacturer" "UNI-ROYAL(Uniroyal Elec)"
-			(at 72.39 54.61 0)
-			(hide yes)
