File: Radio_Receiver_McCormick_Mendoza/MicroSD.kicad_sch (KiCad schematic)
At the start: 8 parts, among them J7 Micro_SD-TF_PUSH

Commit message: Routed antenna and isolated GNDA
Parts:
- J7: footprint 0_Personal:TF-SMD_TF-PUSH -> Reciever_Parts:TF-SMD_TF-PUSH
Changed lines of the file:
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@@
 			)
 		)
-		(property "Footprint" "0_Personal:TF-SMD_TF-PUSH"
+		(property "Footprint" "Reciever_Parts:TF-SMD_TF-PUSH"
 			(at 209.55 83.82 0)
 			(hide yes)
