File: New_Duplicate/Angle_Encoder.kicad_sch (KiCad schematic)
At the start: 8 parts, among them J7 Micro_SD-TF_PUSH

Commit message: New_Duplicate is the new copy working with traces Not everything on the right diagonal is connected
Parts:
- removed C90: 10uF, PCM_JLCPCB:C_0805, symbol PCM_JLCPCB-Capacitors:0805,10uF
- removed C91: 100nF, PCM_JLCPCB:C_0603, symbol PCM_JLCPCB-Capacitors:0603,100nF
- removed J7: Micro_SD-TF_PUSH, 0_Personal:TF-SMD_TF-PUSH, symbol Connector:Micro_SD_Card_Det1
- removed R47, R49, R50, R51, R54: 10kΩ, PCM_JLCPCB:R_0603, symbol PCM_JLCPCB-Resistors:0603,10kΩ
- added C35: 100nF, PCM_JLCPCB:C_0402, symbol PCM_JLCPCB-Capacitors:0402,100nF,(2)
- added C36, C38: 10nF, PCM_JLCPCB:C_0402, symbol PCM_JLCPCB-Capacitors:0402,10nF
- added R7, R8, R9: 10kΩ, PCM_JLCPCB:R_0402, symbol PCM_JLCPCB-Resistors:0402,10kΩ
- added SW1: RotaryEncoder_Switch_MP, Rotary_Encoder:RotaryEncoder_Alps_EC11E-Switch_Vertical_H20mm, symbol Device:RotaryEncoder_Switch_MP
Connections:
- net +3.3V: now also R7.1, R8.1, R9.1
- net GND: now also C35.2, C36.2, C38.2, SW1.C, SW1.MP, SW1.S2
- new net GPIO_A: C36.1, R8.2, SW1.A
- new net GPIO_B: C38.1, R9.2, SW1.B
- new net GPIO_C: C35.1, R7.2, SW1.S1
Other:
- note removed: "If limited for GPIO connectors, card detect is not strictly necessary, and this pin can be NC."
- note removed: "Micro SD Card Slot"
- note removed: "Since SPI mode will be sufficient for this board/project, only 2 of the data lines are used. SDIO would require 4."
