File: New_Duplicate/MicroSD.kicad_sch (KiCad schematic)
At the start: 7 parts, among them SW1 RotaryEncoder_Switch_MP

Commit message: New_Duplicate is the new copy working with traces Not everything on the right diagonal is connected
Parts:
- removed C35: 100nF, PCM_JLCPCB:C_0402, symbol PCM_JLCPCB-Capacitors:0402,100nF,(2)
- removed C36, C38: 10nF, PCM_JLCPCB:C_0402, symbol PCM_JLCPCB-Capacitors:0402,10nF
- removed R7, R8, R9: 10kΩ, PCM_JLCPCB:R_0402, symbol PCM_JLCPCB-Resistors:0402,10kΩ
- removed SW1: RotaryEncoder_Switch_MP, Rotary_Encoder:RotaryEncoder_Alps_EC11E-Switch_Vertical_H20mm, symbol Device:RotaryEncoder_Switch_MP
- added C90: 10uF, PCM_JLCPCB:C_0805, symbol PCM_JLCPCB-Capacitors:0805,10uF
- added C91: 100nF, PCM_JLCPCB:C_0603, symbol PCM_JLCPCB-Capacitors:0603,100nF
- added J7: Micro_SD-TF_PUSH, 0_Personal:TF-SMD_TF-PUSH, symbol Connector:Micro_SD_Card_Det1
- added R47, R49, R50, R51, R54: 10kΩ, PCM_JLCPCB:R_0603, symbol PCM_JLCPCB-Resistors:0603,10kΩ
Connections:
- net +3.3V: now also C90.1, C91.1, J7.4 (VDD), R47.2, R49.2, R50.1, R51.1, R54.2
- net GND: now also C90.2, C91.2, J7.10 (SHIELD), J7.11 (SHIELD), J7.12 (SHIELD), J7.13 (SHIELD), J7.6 (VSS)
- new net CS: J7.2 (DAT3/CS), R51.2
- new net MISO: J7.7 (DAT0/SO), R50.2
- new net MOSI: J7.3 (CMD/SI), R49.1
- new net SD_CD: J7.CD (DET), R54.1
- new net SPI_CK: J7.5 (CLK), R47.1
Other:
- note added: "If limited for GPIO connectors, card detect is not strictly necessary, and this pin can be NC."
- note added: "Micro SD Card Slot"
- note added: "Since SPI mode will be sufficient for this board/project, only 2 of the data lines are used. SDIO would require 4."
